Commit message: its ping!

File: jetsonNano/ros2_ws/src/controller/urdf/robomaster.urdf (robot description, URDF)
Before this commit: robot example_robot, 2 links, 1 joints
Links:
- removed link HCSR04_front_link
- added link PING_sensor_front_link, mass 0.1
Joints:
- joint sensor_joint: child HCSR04_front_link -> PING_sensor_front_link

Commit message: two sensors not parrallel

File: jetsonNano/ros2_ws/src/controller/urdf/robomaster.urdf (robot description, URDF)
Before this commit: robot example_robot, 2 links, 1 joints
Links:
- added link PING_sensor_back_link, mass 0.1
Joints:
- removed joint sensor_joint
- added joint sensor_joint_back: type fixed, parent base_link, child PING_sensor_back_link, origin xyz=-0.15 0 0 rpy=0 0 0
- added joint sensor_joint_front: type fixed, parent base_link, child PING_sensor_front_link, origin xyz=0.15 0 0 rpy=0 0 0

Commit message: works pretty well for both sensors

File: jetsonNano/ros2_ws/src/controller/urdf/robomaster.urdf (robot description, URDF)
Before this commit: robot example_robot, 3 links, 2 joints
Links:
- removed link PING_sensor_back_link
- removed link PING_sensor_front_link
- added link sensor_back, mass 0.1
- added link sensor_front, mass 0.1
Joints:
- joint sensor_joint_back: child PING_sensor_back_link -> sensor_back
- joint sensor_joint_front: child PING_sensor_front_link -> sensor_front
